File: power_module.sch (KiCad schematic (older format))
At the start: 12 parts

Commit message: Added blocks to schematics
Parts:
- removed R? (x6): R, symbol Device:R
- added C? (x4): CP, symbol cooler:CP
- added C? (x2): 100nF, symbol cooler:C
- added C? (x5): C, symbol cooler:C
- added C?: 10nF, symbol cooler:C
- added D?: 1N4004, symbol Device:D
- added D?: MUR120, symbol Device:D
- added J?: Conn_02x05_Male, symbol cooler:Conn_02x05_Male
- added J?: FAN 1, Connectors_JST:JST_VH_B2P-VH-B_2x3.96mm_Vertical, symbol cooler:Conn_01x02_Male
- added J?: FAN 2, Connectors_JST:JST_VH_B2P-VH-B_2x3.96mm_Vertical, symbol cooler:Conn_01x02_Male
- added J?: FAN 3, Connectors_JST:JST_VH_B2P-VH-B_2x3.96mm_Vertical, symbol cooler:Conn_01x02_Male
- added J?: TEC power connector, symbol Connector:Screw_Terminal_01x02
- added K?: SCHRACK420012, Relay_THT:Relay_DPDT_Finder_40.52, symbol Relay:FINDER-41.52
- added L?: 2.2uH, symbol cooler:L_Core_Ferrite
- added Q?: BC547, Package_TO_SOT_THT:TO-92_Inline, symbol Transistor_BJT:BC547
- added Q?: IRF540N, Package_TO_SOT_THT:TO-220-3_Vertical, symbol Transistor_FET:IRF540N
- added R? (x5): 100K, symbol cooler:R
- added R? (x3): 12K, symbol cooler:R
- added R? (x2): 5K6, symbol cooler:R
- added R? (x2): 10K, symbol cooler:R
- added R?: 3K3, symbol cooler:R
- added R?: R, symbol cooler:R
- added R?: 100, symbol cooler:R
- added TP?: TP_12V, symbol Connector:TestPoint
- added TP?: TP_12V_ADC, symbol Connector:TestPoint
- added TP?: TP_GND, symbol Connector:TestPoint
- added TP?: TP_VCC_POWER, symbol Connector:TestPoint
- added TP?: TP_VCC_POWER_ADC, symbol Connector:TestPoint
- added TP?: TP_COLD_HOT_READ, symbol Connector:TestPoint
- added TP?: TP_MOSFET_DRAIN, symbol Connector:TestPoint
- added TP?: TP_PWM_IN, symbol Connector:TestPoint
- added TP?: TP_MOSFET_GATE, symbol Connector:TestPoint
- added U?: UCC27517A, symbol cooler:UCC27517A
- D?: value D -> 1N4004
- J?: footprint (none) -> Cooler:TerminalBlock_bornier-2_P5.08mm
- K?: value FINDER-41.52 -> SCHRACK420012
Connections:
- net labels added: +3.3V, COLD_HOT, COLD_HOT_READ_ADC, DCDC_HIGH_SIDE, DCDC_LOW_SIDE, PWM_IN, TEC_HIGH_SIDE, TEC_LOW_SIDE
- wire segments 30 -> 154
Other:
- note added: "12V -> 1.28V"
- note added: "3.3V\n"
- note added: "BLACK WIRE"
- note added: "CLOSER TO UCC27517 \nVDD AND GND"
- note added: "CLOSER TO \nLOAD"
- note added: "COLD -> BLUE LED ON\nHOT -> YELLOW LED ON"
- note added: "COLD BY DEFAULT"
- note added: "COLD/HOT\nSELECTION\nRELAY"
- note added: "COLD: 1.28V\nHOT: 0.2V\n"
- note added: "FAN\nCONNECTIONS"
- note added: "OFF BY DEFAULT"
- note added: "OPTIONAL LPF"
- note added: "POWER STAGE\nFOR TEC"
- note added: "POWERED ON: 1.28V\nPOWERED OFF: 0V\n"
- note added: "RED WIRE"
- note added: "SIGNAL\nCONNECTOR\n"
- note added: "TODO LIST\n- test points\n- add fans\n- add connectors"
- note removed: "TODO:\n- Add signal connector with control signals\n- Add reverse current relay\n- Add peltier current control circuit\n- Add footprints\n- Generate net\n"

Commit message: Added part numbers except power inductor
Parts:
- removed C?: 100nF, symbol cooler:C
- removed C? (x3): C, symbol cooler:C
- removed C? (x3): CP, symbol cooler:CP
- removed C?: 10nF, symbol cooler:C
- removed D?: 1N4004, symbol Device:D
- removed J?: Power connector, Cooler:TerminalBlock_bornier-2_P5.08mm, symbol Connector:Screw_Terminal_01x02
- removed J?: FAN 2, Connectors_JST:JST_VH_B2P-VH-B_2x3.96mm_Vertical, symbol cooler:Conn_01x02_Male
- removed J?: FAN 3, Connectors_JST:JST_VH_B2P-VH-B_2x3.96mm_Vertical, symbol cooler:Conn_01x02_Male
- removed J?: TEC power connector, symbol Connector:Screw_Terminal_01x02
- removed K?: SCHRACK420012, Relay_THT:Relay_DPDT_Finder_40.52, symbol Relay:FINDER-41.52
- removed Q?: BC547, Package_TO_SOT_THT:TO-92_Inline, symbol Transistor_BJT:BC547
- removed R? (x3): 12K, symbol cooler:R
- removed R? (x2): 5K6, symbol cooler:R
- removed R? (x2): 10K, symbol cooler:R
- removed R?: 3K3, symbol cooler:R
- removed R? (x4): 100K, symbol cooler:R
- removed R?: R, symbol cooler:R
- removed R?: 100, symbol cooler:R
- removed TP?: TP_12V, symbol Connector:TestPoint
- removed TP?: TP_12V_ADC, symbol Connector:TestPoint
- removed TP?: TP_VCC_POWER, symbol Connector:TestPoint
- removed TP?: TP_VCC_POWER_ADC, symbol Connector:TestPoint
- removed TP?: TP_COLD_HOT_READ, symbol Connector:TestPoint
- removed TP?: TP_MOSFET_DRAIN, symbol Connector:TestPoint
- removed TP?: TP_PWM_IN, symbol Connector:TestPoint
- removed TP?: TP_MOSFET_GATE, symbol Connector:TestPoint
- added C? (x3): 10nF, Cooler:C_Rect_L7.0mm_W2.0mm_P5.00mm, symbol cooler:C
- added C?: 100nF, Cooler:C_Rect_L7.0mm_W2.0mm_P5.00mm, symbol cooler:C
- added C? (x2): 220uF, Cooler:CP_Radial_D10.0mm_P5.00mm, symbol cooler:CP
- added C?: 2200uF, Cooler:CP_Radial_D10.0mm_P5.00mm, symbol cooler:CP
- added C? (x2): 100nF, Cooler:C_0603, symbol cooler:C
- added D?: 1N4004, Cooler:D_DO-41_SOD81_P10.16mm_Horizontal, symbol Device:D
- added J?: ScrewTerminal, Cooler:TerminalBlock_bornier-2_P5.08mm, symbol cooler:Screw_Terminal_01x02
- added J?: FAN 2, Cooler:JST_VH_B2P-VH-B_2x3.96mm_Vertical, symbol cooler:Conn_01x02_Male
- added J?: FAN 3, Cooler:JST_VH_B2P-VH-B_2x3.96mm_Vertical, symbol cooler:Conn_01x02_Male
- added J?: TEC Terminal, Cooler:TerminalBlock_bornier-2_P5.08mm, symbol cooler:Screw_Terminal_01x02
- added K?: SCHRACK420012, Cooler:Relay_SPDT_Schrack-RT1-16A-FormC_RM5mm, symbol Relay:FINDER-41.52
- added Q?: BC547, Cooler:TO-92_Inline_Narrow_Oval, symbol Transistor_BJT:BC547
- added R? (x3): 12K, Cooler:R_Axial_DIN0207_L6.3mm_D2.5mm_P10.16mm_Horizontal, symbol cooler:R
- added R? (x6): 100K, Resistors_THT:R_Axial_DIN0207_L6.3mm_D2.5mm_P10.16mm_Horizontal, symbol cooler:R
- added R?: 5K6, Resistors_THT:R_Axial_DIN0207_L6.3mm_D2.5mm_P10.16mm_Horizontal, symbol cooler:R
- added R?: 1, Resistors_THT:R_Axial_DIN0207_L6.3mm_D2.5mm_P10.16mm_Horizontal, symbol cooler:R
- added R? (x2): 100, Resistors_THT:R_Axial_DIN0207_L6.3mm_D2.5mm_P10.16mm_Horizontal, symbol cooler:R
- added R?: 3K3, Cooler:R_Axial_DIN0207_L6.3mm_D2.5mm_P10.16mm_Horizontal, symbol cooler:R
- added TP?: TP_12V, Cooler:TestPoint_Loop_D2.60mm_Drill1.6mm_Beaded, symbol Connector:TestPoint
- added TP?: TP_12V_ADC, Cooler:TestPoint_Loop_D2.60mm_Drill1.6mm_Beaded, symbol Connector:TestPoint
- added TP?: TP_VCC_POWER, Cooler:TestPoint_Loop_D2.60mm_Drill1.6mm_Beaded, symbol Connector:TestPoint
- added TP?: TP_VCC_POWER_ADC, Cooler:TestPoint_Loop_D2.60mm_Drill1.6mm_Beaded, symbol Connector:TestPoint
- added TP?: TP_COLD_HOT_READ, Cooler:TestPoint_Loop_D2.60mm_Drill1.6mm_Beaded, symbol Connector:TestPoint
- added TP?: TP_PWM_IN, Cooler:TestPoint_Loop_D2.60mm_Drill1.6mm_Beaded, symbol Connector:TestPoint
- added TP?: TP_MOSFET_DRAIN, Cooler:TestPoint_Loop_D2.60mm_Drill1.6mm_Beaded, symbol Connector:TestPoint
- added TP?: TP_MOSFET_GATE, Cooler:TestPoint_Loop_D2.60mm_Drill1.6mm_Beaded, symbol Connector:TestPoint
- added TP?: TP_TEC_HIGH_SIDE, Cooler:TestPoint_Loop_D2.60mm_Drill1.6mm_Beaded, symbol Connector:TestPoint
- added TP?: TP_TEC_LOW_SIDE, Cooler:TestPoint_Loop_D2.60mm_Drill1.6mm_Beaded, symbol Connector:TestPoint
- C?: value CP -> 10uF; footprint (none) -> Cooler:CP_Tantalum_Case-B_EIA-3528-21_Reflow; Dielectric type X7R -> tantalium; Farnell Part Number (none) -> 2353056; Manufacturer (none) -> Vishay; Part Number (none) -> 293D106X9025B2TE3; Tolerance 20% -> 10%; Type (none) -> SMD; Voltage 10V -> 25V
- C?: footprint (none) -> Cooler:C_Rect_L7.0mm_W2.0mm_P5.00mm; Farnell Part Number (none) -> 1141777; Manufacturer (none) -> Vishay; Part Number (none) -> K104K15X7RF53H5; Tolerance 1% -> 10%; Type SMD -> TH
- C?: value C -> 10nF; footprint (none) -> Cooler:C_Rect_L7.0mm_W2.0mm_P5.00mm; Dielectric type X7R -> Y5V; Farnell Part Number (none) -> 2309024; Manufacturer (none) -> Multicomp; Part Number (none) -> MC0805Y103M500A5.08MM; Tolerance 1% -> 20%; Type SMD -> TH; Voltage 100V -> 50V
- D?: footprint (none) -> Cooler:D_DO-41_SOD81_P10.16mm_Horizontal; Farnell Part Number (none) -> 9565027; Manufacturer (none) -> Multicomp; Part Number (none) -> 1N4004
- D?: footprint (none) -> Cooler:LED_D5.0mm; Farnell Part Number (none) -> 2449735; MAX Current (none) -> 20 mA; Manufacturer (none) -> Kingbright; Part Number (none) -> L-7083CGDK
- D?: footprint (none) -> Cooler:D_DO-41_SOD81_P10.16mm_Horizontal; Farnell Part Number (none) -> 9557490; Manufacturer (none) -> ON SEMICONDUCTOR; Part Number (none) -> MUR120RLG
- F?: value Fuse 8A -> Fuse Holder; footprint (none) -> Cooler:Fuseholder5x20_horiz_SemiClosed_Casing10x25mm; Farnell Part Number (none) -> 2461161; Manufacturer (none) -> Multicomp; Part Number (none) -> MC000830
- J?: footprint (none) -> Cooler:Multicomp_MC9A12-1034_2x05x2.54mm_Straight
- J?: footprint Connectors_JST:JST_VH_B2P-VH-B_2x3.96mm_Vertical -> Cooler:JST_VH_B2P-VH-B_2x3.96mm_Vertical
- K?: footprint Relay_THT:Relay_DPDT_Finder_40.52 -> Cooler:Relay_SPDT_Schrack-RT1-16A-FormC_RM5mm; Farnell Part Number (none) -> 3103330; Manufacturer (none) -> SCHRACK; Part Number (none) -> RP420012
- Q?: footprint Package_TO_SOT_THT:TO-92_Inline -> Cooler:TO-92_Inline_Narrow_Oval; Farnell Part Number (none) -> 1574381; Manufacturer (none) -> Multicomp; Part Number (none) -> BC547B
- Q?: value IRF540N -> STP60NF06; footprint Package_TO_SOT_THT:TO-220-3_Vertical -> Cooler:TO-220-3_Vertical; Farnell Part Number (none) -> 9803262; Manufacturer (none) -> ST; Part Number (none) -> STP60NF06
- R?: footprint (none) -> Resistors_THT:R_Axial_DIN0207_L6.3mm_D2.5mm_P10.16mm_Horizontal; Farnell Part Number (none) -> 9341129; Manufacturer (none) -> Multicomp; Part Number (none) -> MF25 100K; Power 0.063 W -> 1/4 W; Type SMD 0603 -> THD
- TP?: footprint (none) -> Cooler:TestPoint_Loop_D2.60mm_Drill1.6mm_Beaded; Farnell Part Number (none) -> 2501307; Manufacturer (none) -> Keystone; Part Number (none) -> 5122
- U?: Farnell Part Number (none) -> 2437955; Manufacturer (none) -> TI; Part Number (none) -> UCC27517; Type SOT-23 -> SOT-23-5
Connections:
- wire segments 154 -> 161
Other:
- note added: "6A fuse (protect the TEC)\n"
- note added: "TODO LIST\n- ADD PART AND FOOTPRINTS FOR COIL\n- ADD MECHANICAL PARTS \n- ADD FIDUCIALS & HOLES"
- note removed: "TODO LIST\n- test points\n- add fans\n- add connectors"

Commit message: Modified MOSFET part number selected
Parts:
- Q?: value STP60NF06 -> STP80NF55-06; Farnell Part Number 9803262 -> 1291987; Part Number STP60NF06 -> STP80NF55-06
Changed lines of the file:
@@
 P 6150 4225
 F 0 "Q?" H 6355 4271 50  0000 L CNN
-F 1 "STP60NF06" H 6355 4180 50  0000 L CNN
+F 1 "STP80NF55-06" H 6355 4180 50  0000 L CNN
 F 2 "Cooler:TO-220-3_Vertical" H 6400 4150 50  0001 L CIN
 F 3 "http://www.irf.com/product-info/datasheets/data/irf540n.pdf" H 6150 4225 50  0001 L CNN
-F 4 "STP60NF06" H 6150 4225 50  0001 C CNN "Part Number"
+F 4 "STP80NF55-06" H 6150 4225 50  0001 C CNN "Part Number"
 F 5 "ST" H 6150 4225 50  0001 C CNN "Manufacturer"
-F 6 "9803262" H 6150 4225 50  0001 C CNN "Farnell Part Number"
+F 6 "1291987" H 6150 4225 50  0001 C CNN "Farnell Part Number"
 	1    6150 4225
 	1    0    0    -1
